Commit message: 可以动了，但是动的有问题，可能和惯性矩阵有关

File: install/share/mycar/urdf/mycar.urdf (robot description, URDF)
Before this commit: robot mycar, 4 links, 3 joints
Links:
- added link back_wheel; visual sphere radius=0.025
- added link front_wheel; visual sphere radius=0.025
- added link left_wheel; visual cylinder length=0.015 radius=0.05
- added link right_wheel; visual cylinder length=0.015 radius=0.05
Joints:
- added joint back2link: type continuous, parent base_link, child back_wheel, origin xyz=-0.1 0 -0.075, axis 0 1 0
- added joint front2link: type continuous, parent base_link, child front_wheel, origin xyz=0.1 0 -0.075, axis 0 1 0
- added joint left2link: type continuous, parent base_link, child left_wheel, origin xyz=0 0.1 -0.05, axis 0 1 0
- added joint right2link: type continuous, parent base_link, child right_wheel, origin xyz=0 -0.1 -0.05, axis 0 1 0
- joint link2footprint: origin xyz=0 0 0.05 -> xyz=0 0 0.1
