Commit message: 将万向轮减少至两个，并放置中间，这样就可以原地打转了

File: src/mycar/urdf/color.xacro (robot description, xacro)
@@ -21,5 +21,5 @@
     </material>
     <material name="orange">
-        <color rgba="1.0 0.4235 0.0392 1.0"/>
+        <color rgba="1.0 0.4235 0.0392 0.5"/>
     </material>
     <material name="brown">

File: src/mycar/urdf/move.xacro (robot description, xacro)
@@ -11,6 +11,7 @@
             <left_joint>left2link</left_joint>
             <right_joint>right2link</right_joint>
-            <!-- kinematics -->
+            <!-- 车轮间距 -->
             <wheel_separation>${base_width * 2}</wheel_separation> <!-- 车轮间距 -->
+            <!-- 车轮直径 -->
             <wheel_diameter>${main_wheel_radius * 2}</wheel_diameter><!-- 车轮直径 -->
             <!-- limits -->

File: src/mycar/urdf/my_laser.xacro (robot description, xacro)
@@ -4,4 +4,5 @@
     <xacro:property name="laser_length" value="0.02" />
     <xacro:property name="laser_radius" value="0.02" />
+    <xacro:property name="laser_m" value="0.01" />
     <!-- 雷达宏实现 -->
     <xacro:macro name="add_laser" params="name type">
@@ -22,8 +23,5 @@
             </collision>
             <!-- 惯性矩阵设置 -->
-            <inertial>
-                <mass value="0.2"/>
-                <inertia ixx="0.0122666" ixy="0" ixz="0" iyy="0.0122666" iyz="0" izz="0.02"/>
-            </inertial>
+            <xacro:cylinder_inertial_matrix m="${laser_m}" r="${laser_radius}" h="${laser_length}" />
         </link>
         <joint name="laser_joint${name}" type="fixed">
@@ -37,5 +35,5 @@
             </xacro:if>
             <!-- 设置关节旋转 -->
-            <axis xyz="0 0 1" />
+            <axis xyz="0 0 0" />
         </joint>
     </xacro:macro>

File: src/mycar/urdf/mybase.xacro (robot description, xacro)
@@ -14,11 +14,17 @@
     <xacro:property name="base_width" value="0.2" />
     <xacro:property name="base_depth" value="0.1" />
-    <xacro:property name="base_up" value="0.03" /> <!-- 小车地盘离地距离 -->
+    <xacro:property name="base_up" value="0.02" /> <!-- 小车地盘离地距离 -->
     <xacro:property name="base_center_up" value="${base_depth/2 + base_up}" /> <!-- 小车中心点离地距离 -->
+    <xacro:property name="base_m" value="0.5" /> <!-- 地盘重量 -->
     <!-- 主动轮相关参数 -->
-    <xacro:property name="main_wheel_radius" value="0.05"  />
+    <xacro:property name="main_wheel_radius" value="0.03"  />
     <xacro:property name="main_wheel_length" value="0.015" />
+    <xacro:property name="main_wheel_m" value="0.1" />
     <!-- 从动轮相关参数 -->
     <xacro:property name="sub_wheel_radius" value="0.015"  />
+    <xacro:property name="sub_wheel_length" value="0.015" />
+    <xacro:property name="sub_wheel_m" value="0.1"  />
+    <xacro:property name="sub_wheel_offset1" value="0.05"  />
+    <xacro:property name="sub_wheel_offset2" value="0.02"  />
     <!-- base link 小车中心的位置-->
     <link name="base_link">
@@ -40,8 +46,5 @@
         </collision>
         <!-- 惯性矩阵设置 -->
-        <inertial>
-            <mass value="0.2"/>
-            <inertia ixx="0.0122666" ixy="0" ixz="0" iyy="0.0122666" iyz="0" izz="0.02"/>
-        </inertial>
+        <xacro:Box_inertial_matrix m="${base_m}" l="${base_length}" w="${base_width}" h="${base_depth}" />
     </link>
     <!-- 使小车距离地面上方0.05M -->
@@ -59,5 +62,5 @@
                 <origin xyz="0 0 0" rpy="1.5708 0 0"/>
                 <geometry>
-                    <cylinder radius="0.05" length="0.015"></cylinder>
+                    <cylinder radius="${main_wheel_radius}" length="${main_wheel_length}"></cylinder>
                 </geometry>
                 <material name="grey"/>
@@ -67,12 +70,9 @@
                 <origin xyz="0 0 0" rpy="1.5708 0 0"/>
                 <geometry>
-                    <cylinder radius="0.05" length="0.015"></cylinder>
+                    <cylinder radius="${main_wheel_radius}" length="${main_wheel_length}"></cylinder>
                 </geometry>
             </collision>
             <!-- 惯性矩阵设置 -->
-            <inertial>
-                <mass value="0.2"/>
-                <inertia ixx="0.0122666" ixy="0" ixz="0" iyy="0.0122666" iyz="0" izz="0.02"/>
-            </inertial>
+            <xacro:cylinder_inertial_matrix m="${main_wheel_m}" r="${main_wheel_radius}" h="${main_wheel_length}" />
         </link>
         <joint name="${name}2link" type="continuous">
@@ -100,4 +100,7 @@
             <visual>
                 <origin xyz="0 0 0" rpy="0 0 0"/>
+                <!-- <geometry>
+                    <cylinder radius="${sub_wheel_radius}" length="${sub_wheel_length}"></cylinder>
+                </geometry> -->
                 <geometry>
                     <sphere radius="${sub_wheel_radius}"/>
@@ -112,8 +115,5 @@
             </collision>
             <!-- 惯性矩阵设置 -->
-            <inertial>
-                <mass value="0.2"/>
-                <inertia ixx="0.0122666" ixy="0" ixz="0" iyy="0.0122666" iyz="0" izz="0.02"/>
-            </inertial>
+            <xacro:sphere_inertial_matrix m="${sub_wheel_m}" r="${sub_wheel_radius}" />
         </link>
         <joint name="wheel${name}_joint" type="continuous">
@@ -121,25 +121,31 @@
             <child link="wheel${name}" />
             <!-- 左上 -->
-            <xacro:if value="${pos == 'q'}">
+            <!-- <xacro:if value="${pos == 'q'}">
                 <origin xyz="${base_length/2} ${base_width/2} ${-(base_center_up - sub_wheel_radius)}" />
+            </xacro:if> -->
+            <!-- 右上 -->
+            <!-- <xacro:if value="${pos == 'e'}">
+                <origin xyz="${-base_length/2} ${base_width/2 } ${-(base_center_up - sub_wheel_radius)}" />
+            </xacro:if> -->
+            <!-- 左下 -->
+            <!-- <xacro:if value="${pos == 'z'}">
+                <origin xyz="${base_length/2} ${-base_width/2 } ${-(base_center_up - sub_wheel_radius)}" />
+            </xacro:if> -->
+            <!-- 右下 -->
+            <!-- <xacro:if value="${pos == 'c'}">
+                <origin xyz="${-base_length/2} ${-base_width/2 } ${-(base_center_up - sub_wheel_radius)}" />
+            </xacro:if> -->
+            <xacro:if value="${pos == 'z'}">
+                <origin xyz="${base_length/2} 0 ${-(base_center_up - sub_wheel_radius)}" />
             </xacro:if>
-            <!-- 右上 -->
-            <xacro:if value="${pos == 'e'}">
-                <origin xyz="${-base_length/2} ${base_width/2} ${-(base_center_up - sub_wheel_radius)}" />
+            <xacro:if value="${pos == 'c'}">
+                <origin xyz="${-base_length/2} 0 ${-(base_center_up - sub_wheel_radius)}" />
             </xacro:if>
-            <!-- 左下 -->
-            <xacro:if value="${pos == 'z'}">
-                <origin xyz="${base_length/2} ${-base_width/2} ${-(base_center_up - sub_wheel_radius)}" />
-            </xacro:if>
-            <!-- 右下 -->
-            <xacro:if value="${pos == 'c'}">
-                <origin xyz="${-base_length/2} ${-base_width/2} ${-(base_center_up - sub_wheel_radius)}" />
-            </xacro:if>
-            <axis xyz="0 1 0" />
+            <axis xyz="0 1 1" />
         </joint>
     </xacro:macro>
     <!-- 四个万向轮实现 -->
-    <xacro:add_sub_wheel name="1" pos="q"/>
-    <xacro:add_sub_wheel name="2" pos="e"/>
+    <!-- <xacro:add_sub_wheel name="1" pos="q"/>
+    <xacro:add_sub_wheel name="2" pos="e"/>  -->
     <xacro:add_sub_wheel name="3" pos="z"/>
     <xacro:add_sub_wheel name="4" pos="c"/>

File: src/mycar/urdf/mycar.xacro (robot description, xacro)
@@ -4,4 +4,5 @@
     <!-- <test>${pi}</test> -->
     <xacro:include filename="color.xacro"/>
+    <xacro:include filename="inertial_matrix.xacro"/>
     <xacro:include filename="mybase.xacro"/>
     <xacro:include filename="my_laser.xacro"/>
