Commit message: 新增imu，slma建图生成静态地图

File: src/mycar/urdf/my_laser.xacro (robot description, xacro)
@@ -47,3 +47,51 @@
         <material>Gazebo/Black</material>
     </gazebo>
+    <gazebo reference="laser_link1">
+        <sensor name="laser_sensor" type="ray">
+            <always_on>true</always_on>
+            <visualize>true</visualize>
+            <pose>-0.032 0 0.171 0 0 0</pose>
+            <update_rate>5</update_rate>
+            <ray>
+                <!-- 激光雷达扫描参数设置 -->
+                <scan>
+                    <horizontal>
+                        <!-- 360条光束（扫描密度） -->
+                        <samples>360</samples>
+                        <!-- 采样,每n条光束有一条测量距离，为了减轻仿真压力 -->
+                        <resolution>1</resolution>
+                        <!-- 扫描范围，单位弧度 -->
+                        <min_angle>${-pi/2}</min_angle>
+                        <max_angle>${pi}</max_angle>
+                    </horizontal>
+                </scan>
+                <!-- 雷达检测范围和精度 -->
+                <range>
+                    <!-- 10厘米以内的探测不到 -->
+                    <min>0.100000</min>
+                    <!-- 5米之外的探测不到 -->
+                    <max>5.0</max>
+                    <!-- 探测精度为1厘米 -->
+                    <resolution>0.01</resolution>
+                </range>
+                <!-- 添加高斯噪音（贴近真实的环境） -->
+                <noise>
+                    <type>gaussian</type>
+                    <mean>0.0</mean>
+                    <stddev>0.01</stddev>
+                </noise>
+            </ray>
+            <plugin name="laserscan" filename="libgazebo_ros_ray_sensor.so">
+                <ros>
+                    <!-- <namespace>/tb3</namespace> -->
+                    <!-- 话题发布 -->
+                    <remapping>~/out:=/scan</remapping>
+                </ros>
+                <!-- 雷达消息类型 -->
+                <output_type>sensor_msgs/LaserScan</output_type>
+                <!-- 关联到哪个link -->
+                <frame_name>laser_link1</frame_name>
+            </plugin>
+        </sensor>
+    </gazebo>
 </robot>

File: src/mycar/urdf/mybase.xacro (robot description, xacro)
@@ -11,20 +11,21 @@
     </link>
     <!-- 小车地盘相关参数 -->
-    <xacro:property name="base_length" value="0.3" />
-    <xacro:property name="base_width" value="0.2" />
-    <xacro:property name="base_depth" value="0.1" />
-    <xacro:property name="base_up" value="0.02" /> <!-- 小车地盘离地距离 -->
+    <xacro:property name="base_length" value="1.21" />
+    <xacro:property name="base_width" value="0.738" />
+    <xacro:property name="base_depth" value="0.35" />
+    <xacro:property name="base_up" value="0.028" /> <!-- 小车地盘离地距离 -->
     <xacro:property name="base_center_up" value="${base_depth/2 + base_up}" /> <!-- 小车中心点离地距离 -->
     <xacro:property name="base_m" value="0.5" /> <!-- 地盘重量 -->
     <!-- 主动轮相关参数 -->
-    <xacro:property name="main_wheel_radius" value="0.03"  />
-    <xacro:property name="main_wheel_length" value="0.015" />
+    <xacro:property name="main_wheel_radius" value="0.10"  />
+    <xacro:property name="main_wheel_length" value="0.06" />
     <xacro:property name="main_wheel_m" value="0.1" />
     <!-- 从动轮相关参数 -->
-    <xacro:property name="sub_wheel_radius" value="0.015"  />
-    <xacro:property name="sub_wheel_length" value="0.015" />
+    <xacro:property name="sub_wheel_radius" value="0.05"  />
+    <xacro:property name="sub_wheel_length" value="0.055" />
     <xacro:property name="sub_wheel_m" value="0.1"  />
-    <xacro:property name="sub_wheel_offset1" value="0.05"  />
-    <xacro:property name="sub_wheel_offset2" value="0.02"  />
+    <xacro:property name="wheel_offset_up" value="0.102"  />
+    <xacro:property name="main_wheel_offset_left" value="0.039"  />
+    <xacro:property name="sub_wheel_offset_left" value="0.091"  />
     <!-- base link 小车中心的位置-->
     <link name="base_link">
@@ -83,8 +84,8 @@
             Z 方向：baselink距离地面的高度 - 车轮半径 -->
             <xacro:if value="${type == 'left'}">
-                <origin xyz="0 ${base_width/2} ${-(base_center_up - main_wheel_radius)}" />
+                <origin xyz="0 ${base_width/2 - main_wheel_offset_left} ${-(base_center_up - main_wheel_radius)}" />
             </xacro:if>
             <xacro:if value="${type == 'right'}">
-                <origin xyz="0 ${-base_width/2} ${-(base_center_up - main_wheel_radius)}" />
+                <origin xyz="0 ${-base_width/2 + main_wheel_offset_left} ${-(base_center_up - main_wheel_radius)}" />
             </xacro:if>
             <!-- 绕Y轴转动 -->
@@ -122,23 +123,23 @@
             <!-- 左上 -->
             <!-- <xacro:if value="${pos == 'q'}">
-                <origin xyz="${base_length/2} ${base_width/2} ${-(base_center_up - sub_wheel_radius)}" />
+                <origin xyz="${base_length/2 - wheel_offset_up} ${base_width/2 - sub_wheel_offset_left} ${-(base_center_up - sub_wheel_radius)}" />
             </xacro:if> -->
             <!-- 右上 -->
             <!-- <xacro:if value="${pos == 'e'}">
-                <origin xyz="${-base_length/2} ${base_width/2 } ${-(base_center_up - sub_wheel_radius)}" />
+                <origin xyz="${-base_length/2 + wheel_offset_up} ${base_width/2 - sub_wheel_offset_left} ${-(base_center_up - sub_wheel_radius)}" />
             </xacro:if> -->
             <!-- 左下 -->
             <!-- <xacro:if value="${pos == 'z'}">
-                <origin xyz="${base_length/2} ${-base_width/2 } ${-(base_center_up - sub_wheel_radius)}" />
+                <origin xyz="${base_length/2 - wheel_offset_up} ${-base_width/2 + sub_wheel_offset_left} ${-(base_center_up - sub_wheel_radius)}" />
             </xacro:if> -->
             <!-- 右下 -->
             <!-- <xacro:if value="${pos == 'c'}">
-                <origin xyz="${-base_length/2} ${-base_width/2 } ${-(base_center_up - sub_wheel_radius)}" />
+                <origin xyz="${-base_length/2 + wheel_offset_up} ${-base_width/2 + sub_wheel_offset_left} ${-(base_center_up - sub_wheel_radius)}" />
             </xacro:if> -->
             <xacro:if value="${pos == 'z'}">
-                <origin xyz="${base_length/2} 0 ${-(base_center_up - sub_wheel_radius)}" />
+                <origin xyz="${base_length/2 - wheel_offset_up} 0 ${-(base_center_up - sub_wheel_radius)}" />
             </xacro:if>
             <xacro:if value="${pos == 'c'}">
-                <origin xyz="${-base_length/2} 0 ${-(base_center_up - sub_wheel_radius)}" />
+                <origin xyz="${-base_length/2 + wheel_offset_up} 0 ${-(base_center_up - sub_wheel_radius)}" />
             </xacro:if>
             <axis xyz="0 1 1" />

File: src/mycar/urdf/mycar.xacro (robot description, xacro)
@@ -7,4 +7,5 @@
     <xacro:include filename="mybase.xacro"/>
     <xacro:include filename="my_laser.xacro"/>
+    <xacro:include filename="my_imu.xacro"/>
     <!-- 集成运动控制 -->
     <xacro:include filename="move.xacro"/>
