Commit message: 改为四个雷达，微调摄像头位置

File: src/mycar/urdf/my_camera.xacro (robot description, xacro)
@@ -7,5 +7,5 @@
     <xacro:property name="camera_x" value="${base_length / 2}" /> <!-- 摄像头安装的x坐标 -->
     <xacro:property name="camera_y" value="0.0" /> <!-- 摄像头安装的y坐标 -->
-    <xacro:property name="camera_z" value="${base_depth / 2 + camera_height / 2}" /> <!-- 摄像头安装的z坐标:底盘高度 / 2 + 摄像头高度 / 2  -->
+    <xacro:property name="camera_z" value="${0.192 - base_depth / 2 }" /> <!-- 摄像头安装的z坐标:底盘高度 / 2 + 摄像头高度 / 2  -->
     <xacro:property name="camera_m" value="0.01" /> <!-- 摄像头质量 -->
     <link name="camera_link">

File: src/mycar/urdf/my_ultrasound.xacro (robot description, xacro)
@@ -28,9 +28,15 @@
             <parent link="base_link" />
             <child link="ultra_link${name}" />
-            <xacro:if value="${type == 'head'}">
-                <origin xyz="${base_length/2 + ultra_radius} 0 0" />
+            <xacro:if value="${type == 'head_left'}">
+                <origin xyz="${base_length/2 + ultra_radius} 0.149 0 "/>
             </xacro:if>
-            <xacro:if value="${type == 'tail'}">
-                <origin xyz="${-base_length/2 - ultra_radius} 0 0" />
+            <xacro:if value="${type == 'tail_left'}">
+                <origin xyz="${-base_length/2 - ultra_radius} 0.149 0" />
+            </xacro:if>
+            <xacro:if value="${type == 'head_right'}">
+                <origin xyz="${base_length/2 + ultra_radius} -0.149 0" />
+            </xacro:if>
+            <xacro:if value="${type == 'tail_right'}">
+                <origin xyz="${-base_length/2 - ultra_radius} -0.149 0" />
             </xacro:if>
             <!-- 设置关节旋转 -->
@@ -38,7 +44,9 @@
         </joint>
     </xacro:macro>
-    <!-- 调用宏添加雷达(type这个参数不能是数字) -->
-    <xacro:add_ultra name="1" type="head"/>
-    <xacro:add_ultra name="2" type="tail"/>
+    <!-- 调用宏(type这个参数不能是数字) -->
+    <xacro:add_ultra name="1" type="head_left"/>
+    <xacro:add_ultra name="2" type="head_right"/>
+    <xacro:add_ultra name="3" type="tail_left"/>
+    <xacro:add_ultra name="4" type="tail_right"/>
     <!-- ～～～～～～～～～～～～～gazebo～～～～～～～～～～～～～～～～～ -->
     <xacro:macro name="add_ultra_gazebo" params="name type">
@@ -55,9 +63,9 @@
                             <samples>10</samples>
                             <resolution>1</resolution>
-                            <xacro:if value="${type == 'head'}">
+                            <xacro:if value="${type == 'head_left' or type == 'head_right'}">
                                 <min_angle>-0.087</min_angle>
                                 <max_angle>0.087</max_angle>
                             </xacro:if>
-                            <xacro:if value="${type == 'tail'}">
+                            <xacro:if value="${type == 'tail_left' or type == 'tail_right'}">
                                 <min_angle>${-0.087 + pi}</min_angle>
                                 <max_angle>${0.087 + pi}</max_angle>
@@ -102,5 +110,7 @@
         </gazebo>
     </xacro:macro>
-    <xacro:add_ultra_gazebo name="1" type="head"/>
-    <xacro:add_ultra_gazebo name="2" type="tail"/>
+    <xacro:add_ultra_gazebo name="1" type="head_left"/>
+    <xacro:add_ultra_gazebo name="2" type="head_right"/>
+    <xacro:add_ultra_gazebo name="3" type="tail_left"/>
+    <xacro:add_ultra_gazebo name="4" type="tail_right"/>
 </robot>
