Commit message: 通过启动 bringup_launch.py 启动整个Nav2 ，目前实现了地图的加载，接下来实现代价地图的显示，以及如何导航到目标点

File: src/mycar/urdf/move.xacro (robot description, xacro)
@@ -8,4 +8,8 @@
                     <remapping>odom:=odom</remapping>
                 </ros> -->
+                <remapping>/tf:=tf</remapping>
+            <ros>
+                <remapping>odom:=odom</remapping>
+            </ros>
             <!-- wheels -->
             <left_joint>left2link</left_joint>
@@ -25,4 +29,5 @@
             <robot_base_frame>base_footprint</robot_base_frame>
         </plugin>
+        <!-- 这个去掉貌似也没啥影响 -->
         <plugin name="car_joint_state" filename="libgazebo_ros_joint_state_publisher.so">
             <ros>
@@ -32,5 +37,4 @@
             <joint_name>left2link</joint_name>
             <joint_name>right2link</joint_name>
-            <!-- <joint_name>caster_joint</joint_name> -->
         </plugin>
     </gazebo>

File: src/mycar/urdf/mycar.urdf (robot description, URDF)
Before this commit: robot mycar, 8 links, 7 joints
Links:
- removed link back_wheel
- removed link front_wheel
- added link camera_link, mass 0.01; collision box size=0.01 0.025 0.025; visual box size=0.01 0.025 0.025
- added link imu_link, mass 0.1; collision box size=0.1 0.1 0.1; visual box size=0.1 0.1 0.1
- added link ultra_link1, mass 0.01; collision cylinder length=0.02 radius=0.02; visual cylinder length=0.02 radius=0.02
- added link ultra_link2, mass 0.01; collision cylinder length=0.02 radius=0.02; visual cylinder length=0.02 radius=0.02
- added link ultra_link3, mass 0.01; collision cylinder length=0.02 radius=0.02; visual cylinder length=0.02 radius=0.02
- added link ultra_link4, mass 0.01; collision cylinder length=0.02 radius=0.02; visual cylinder length=0.02 radius=0.02
- added link wheel3, mass 0.1; collision sphere radius=0.05; visual sphere radius=0.05
- added link wheel4, mass 0.1; collision sphere radius=0.05; visual sphere radius=0.05
- link base_link: mass None -> 0.5; geometry collision box size=1.21 0.738 0.35; visual box size=1.21 0.738 0.35
- link laser_link1: mass None -> 0.01; geometry collision cylinder length=0.02 radius=0.02; visual cylinder length=0.02 radius=0.02
- link laser_link2: mass None -> 0.01; geometry collision cylinder length=0.02 radius=0.02; visual cylinder length=0.02 radius=0.02
- link left_wheel: mass None -> 0.1; geometry collision cylinder length=0.06 radius=0.1; visual cylinder length=0.06 radius=0.1
- link right_wheel: mass None -> 0.1; geometry collision cylinder length=0.06 radius=0.1; visual cylinder length=0.06 radius=0.1
Joints:
- removed joint back2link
- removed joint front2link
- added joint camera_joint: type fixed, parent base_link, child camera_link, origin xyz=0.605 0.0 0.017000000000000015
- added joint imu_joint: type fixed, parent base_link, child imu_link, origin xyz=0 0 0.01
- added joint ultra_joint1: type fixed, parent base_link, child ultra_link1, origin xyz=0.625 0.149 0 , axis 0 0 0
- added joint ultra_joint2: type fixed, parent base_link, child ultra_link2, origin xyz=0.625 -0.149 0, axis 0 0 0
- added joint ultra_joint3: type fixed, parent base_link, child ultra_link3, origin xyz=-0.625 0.149 0, axis 0 0 0
- added joint ultra_joint4: type fixed, parent base_link, child ultra_link4, origin xyz=-0.625 -0.149 0, axis 0 0 0
- added joint wheel3_joint: type continuous, parent base_link, child wheel3, origin xyz=0.503 0 -0.15299999999999997, axis 0 1 1
- added joint wheel4_joint: type continuous, parent base_link, child wheel4, origin xyz=-0.503 0 -0.15299999999999997, axis 0 1 1
- joint laser_joint1: axis 0 0 1 -> 0 0 0; origin xyz=0.15 0.1 0.05 -> xyz=0.605 0.369 0.175; type continuous -> fixed
- joint laser_joint2: axis 0 0 1 -> 0 0 0; origin xyz=-0.15 -0.1 0.05 -> xyz=-0.605 -0.369 0.175; type continuous -> fixed
- joint left2link: origin xyz=0 0.1 -0.05 -> xyz=0 0.33 -0.10299999999999998
- joint link2footprint: origin xyz=0 0 0.1 -> xyz=0 0 0.20299999999999999
- joint right2link: origin xyz=0 -0.1 -0.05 -> xyz=0 -0.33 -0.10299999999999998

Commit message: 速度已提到最大的设置速度1.5

File: src/mycar/urdf/move.xacro (robot description, xacro)
@@ -20,6 +20,6 @@
             <wheel_diameter>${main_wheel_radius * 2}</wheel_diameter><!-- 车轮直径 -->
             <!-- limits -->
-            <max_wheel_torque>20</max_wheel_torque>
-            <max_wheel_acceleration>0.5</max_wheel_acceleration>
+            <max_wheel_torque>70</max_wheel_torque>
+            <max_wheel_acceleration>5</max_wheel_acceleration>
             <!-- output -->
             <publish_odom>true</publish_odom>

File: src/mycar/urdf/my_laser.xacro (robot description, xacro)
@@ -51,6 +51,6 @@
             <always_on>true</always_on>
             <visualize>true</visualize>
-            <pose>-0.032 0 0.171 0 0 0</pose>
-            <update_rate>5</update_rate>
+            <pose>0 0 0 0 0 0</pose>
+            <update_rate>5.5</update_rate>
             <ray>
                 <!-- 激光雷达扫描参数设置 -->

File: src/mycar/urdf/mybase.xacro (robot description, xacro)
@@ -3,10 +3,4 @@
     <!-- 地平面的位置   -->
     <link name="base_footprint">
-        <visual>
-        <origin xyz="0 0 0.0" rpy="0 0 0"/>
-        <geometry>
-            <box size="0.00001 0.00001 0.00001"></box>
-        </geometry>
-        </visual>
     </link>
     <!-- 小车地盘相关参数 -->
